File: pcb/pcb.kicad_sch (KiCad schematic)
At the start: 38 parts, among them J1 Conn_01x04_Pin, J2 Conn_01x06_Pin, U1 XIAO-ESP32-C5-DIP, U10 XIAO-ESP32-C5-DIP, U11 XIAO-ESP32-C5-DIP, U12 XIAO-ESP32-C5-DIP, U13 XIAO-ESP32-C5-DIP, U14 XIAO-ESP32-C5-DIP, U15 XIAO-ESP32-C5-DIP, U18 XIAO-ESP32-C5-DIP, U19 LD1117V33, U2 XIAO-ESP32-C5-DIP, U3 XIAO-ESP32-C5-DIP, U4 XIAO-ESP32-C5-DIP, U5 XIAO-ESP32-C5-DIP, U6 XIAO-ESP32-C5-DIP, U7 XIAO-ESP32-C5-DIP, U8 XIAO-ESP32-C5-DIP, U9 XIAO-ESP32-C5-DIP

Commit message: add capacitors to i/o of LD1117
Parts:
- added C1: 100nF, Capacitor_THT:C_Disc_D5.0mm_W2.5mm_P2.50mm, symbol Device:C
- added C2: 10uF, Capacitor_THT:C_Disc_D5.0mm_W2.5mm_P2.50mm, symbol Device:C
Connections:
- net +5V: now also C1.2; no longer U19.3 (VI)
- net at J2.6 (Pin_6), R1.2: now also C2.1; no longer U19.2 (VO)
- new net: C2.2, U19.2 (VO)
- new net: C1.1, U19.3 (VI)
Changed lines of the file:
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@@
 	)
 	(junction
+		(at 143.51 215.9)
+		(diameter 0)
+		(color 0 0 0 0)
+	)
+	(junction
 		(at 87.63 48.26)
 		(diameter 0)
@@
 	)
 	(junction
-		(at 143.51 215.9)
-		(diameter 0)
-		(color 0 0 0 0)
-	)
-	(junction
 		(at 87.63 212.09)
 		(diameter 0)
@@
 	(wire
 		(pts
-			(xy 143.51 224.79) (xy 139.7 224.79)
-		)
-		(stroke
-			(width 0)
-			(type default)
-		)
-	)
-	(wire
-		(pts
 			(xy 87.63 212.09) (xy 87.63 205.74)
 		)
@@
 	(wire
 		(pts
+			(xy 116.84 238.76) (xy 116.84 232.41)
+		)
+		(stroke
+			(width 0)
+			(type default)
+		)
+	)
+	(wire
+		(pts
 			(xy 102.87 308.61) (xy 119.38 308.61)
 		)
@@
 	(wire
 		(pts
+			(xy 116.84 224.79) (xy 124.46 224.79)
+		)
+		(stroke
+			(width 0)
+			(type default)
+		)
+	)
+	(wire
+		(pts
 			(xy 76.2 157.48) (xy 73.66 157.48)
 		)
@@
 	(wire
 		(pts
-			(xy 143.51 215.9) (xy 143.51 224.79)
-		)
-		(stroke
-			(width 0)
-			(type default)
-		)
-	)
-	(wire
-		(pts
 			(xy 88.9 269.24) (xy 74.93 269.24)
 		)
@@
 	(wire
 		(pts
+			(xy 143.51 215.9) (xy 143.51 217.17)
+		)
+		(stroke
+			(width 0)
+			(type default)
+		)
+	)
+	(wire
+		(pts
 			(xy 87.63 90.17) (xy 87.63 88.9)
 		)
@@
 	(wire
 		(pts
-			(xy 119.38 224.79) (xy 124.46 224.79)
-		)
-		(stroke
-			(width 0)
-			(type default)
-		)
-	)
-	(wire
-		(pts
 			(xy 152.4 303.53) (xy 147.32 303.53)
 		)
@@
 	(wire
 		(pts
+			(xy 139.7 224.79) (xy 143.51 224.79)
+		)
+		(stroke
+			(width 0)
+			(type default)
+		)
+	)
+	(wire
+		(pts
 			(xy 82.55 238.76) (xy 87.63 238.76)
 		)
@@
 	(wire
 		(pts
+			(xy 119.38 238.76) (xy 116.84 238.76)
+		)
+		(stroke
+			(width 0)
+			(type default)
+		)
+	)
+	(wire
+		(pts
 			(xy 180.34 90.17) (xy 246.38 90.17)
 		)
@@
 	(symbol
 		(lib_id "power:+5V")
-		(at 119.38 224.79 0)
+		(at 119.38 238.76 0)
 		(unit 1)
 		(body_style 1)
@@
 		(fields_autoplaced yes)
 		(property "Reference" "#PWR07"
-			(at 119.38 228.6 0)
+			(at 119.38 242.57 0)
 			(hide yes)
 			(show_name no)
@@
 		)
 		(property "Value" "+5V"
-			(at 119.38 219.71 0)
+			(at 119.38 233.68 0)
 			(show_name no)
 			(do_not_autoplace no)
@@
 		)
 		(property "Footprint" ""
-			(at 119.38 224.79 0)
+			(at 119.38 238.76 0)
 			(hide yes)
 			(show_name no)
@@
 		)
 		(property "Datasheet" ""
-			(at 119.38 224.79 0)
+			(at 119.38 238.76 0)
 			(hide yes)
 			(show_name no)
@@
 		)
 		(property "Description" "Power symbol creates a global label with name \"+5V\""
-			(at 119.38 224.79 0)
+			(at 119.38 238.76 0)
 			(hide yes)
 			(show_name no)
@@
 	)
 	(symbol
+		(lib_id "Device:C")
+		(at 116.84 228.6 0)
+		(unit 1)
+		(body_style 1)
+		(exclude_from_sim no)
+		(in_bom yes)
+		(on_board yes)
+		(in_pos_files yes)
+		(dnp no)
+		(fields_autoplaced yes)
+		(property "Reference" "C1"
+			(at 120.65 227.3299 0)
+			(show_name no)
+			(do_not_autoplace no)
+			(effects
+				(font
+					(size 1.27 1.27)
+				)
+				(justify left)
+			)
+		)
+		(property "Value" "100nF"
+			(at 120.65 229.8699 0)
+			(show_name no)
+			(do_not_autoplace no)
+			(effects
+				(font
+					(size 1.27 1.27)
+				)
+				(justify left)
+			)
+		)
+		(property "Footprint" "Capacitor_THT:C_Disc_D5.0mm_W2.5mm_P2.50mm"
+			(at 117.8052 232.41 0)
+			(hide yes)
+			(show_name no)
+			(do_not_autoplace no)
+			(effects
+				(font
+					(size 1.27 1.27)
+				)
+			)
+		)
+		(property "Datasheet" ""
+			(at 116.84 228.6 0)
+			(hide yes)
+			(show_name no)
+			(do_not_autoplace no)
+			(effects
+				(font
+					(size 1.27 1.27)
+				)
+			)
+		)
+		(property "Description" "Unpolarized capacitor"
+			(at 116.84 228.6 0)
+			(hide yes)
+			(show_name no)
+			(do_not_autoplace no)
+			(effects
+				(font
+					(size 1.27 1.27)
+				)
+			)
+		)
+		(pin "2"
+		)
+		(pin "1"
+		)
+		(instances
+			(project "pcb"
+				(path "/177b52ef-cce2-4dab-a936-75649664352c"
+					(reference "C1")
+					(unit 1)
+				)
+			)
+		)
+	)
+	(symbol
 		(lib_id "power:+5V")
 		(at 142.24 25.4 0)
@@
 					(unit 1)
 				)
+			)
+		)
+	)
+	(symbol
+		(lib_id "Device:C")
+		(at 143.51 220.98 0)
+		(unit 1)
+		(body_style 1)
+		(exclude_from_sim no)
+		(in_bom yes)
+		(on_board yes)
+		(in_pos_files yes)
+		(dnp no)
+		(fields_autoplaced yes)
+		(property "Reference" "C2"
+			(at 147.32 219.7099 0)
+			(show_name no)
+			(do_not_autoplace no)
+			(effects
+				(font
+					(size 1.27 1.27)
+				)
+				(justify left)
+			)
+		)
+		(property "Value" "10uF"
+			(at 147.32 222.2499 0)
+			(show_name no)
+			(do_not_autoplace no)
+			(effects
+				(font
+					(size 1.27 1.27)
+				)
+				(justify left)
+			)
+		)
+		(property "Footprint" "Capacitor_THT:C_Disc_D5.0mm_W2.5mm_P2.50mm"
+			(at 144.4752 224.79 0)
+			(hide yes)
+			(show_name no)
+			(do_not_autoplace no)
+			(effects
+				(font
+					(size 1.27 1.27)
+				)
+			)
+		)
+		(property "Datasheet" ""
+			(at 143.51 220.98 0)
+			(hide yes)
+			(show_name no)
+			(do_not_autoplace no)
+			(effects
+				(font
+					(size 1.27 1.27)
+				)
+			)
+		)
+		(property "Description" "Unpolarized capacitor"
+			(at 143.51 220.98 0)
+			(hide yes)
+			(show_name no)
+			(do_not_autoplace no)
+			(effects
+				(font
+					(size 1.27 1.27)
+				)
+			)
+		)
+		(pin "1"
+		)
+		(pin "2"
+		)
+		(instances
+			(project "pcb"
+				(path "/177b52ef-cce2-4dab-a936-75649664352c"
+					(reference "C2")
+					(unit 1)
+				)
