File: pcb/pcb.kicad_sch (KiCad schematic)
At the start: 40 parts, among them J1 Conn_01x04_Pin, J2 Conn_01x06_Pin, U1 XIAO-ESP32-C5-DIP, U10 XIAO-ESP32-C5-DIP, U11 XIAO-ESP32-C5-DIP, U12 XIAO-ESP32-C5-DIP, U13 XIAO-ESP32-C5-DIP, U14 XIAO-ESP32-C5-DIP, U15 XIAO-ESP32-C5-DIP, U18 XIAO-ESP32-C5-DIP, U19 LD1117V33, U2 XIAO-ESP32-C5-DIP, U3 XIAO-ESP32-C5-DIP, U4 XIAO-ESP32-C5-DIP, U5 XIAO-ESP32-C5-DIP, U6 XIAO-ESP32-C5-DIP, U7 XIAO-ESP32-C5-DIP, U8 XIAO-ESP32-C5-DIP, U9 XIAO-ESP32-C5-DIP

Commit message: add CS labels
Parts:
- U17: renamed from U16; value (none) -> ESP32-S3 DevKitC-A
- renumbered U18 to U15, U15 to U16, U19 to U18
Connections:
- net CS 3: now reaches R4.2, U17.6 (GPIO6), U3.3 (GPIO25_D2)
- net CS 11: now reaches R12.2, U11.3 (GPIO25_D2), U17.29 (GPIO41)
- net CS 14: now reaches R15.2, U14.3 (GPIO25_D2), U17.40 (GPIO21)
- net CS 9: now reaches R10.2, U17.27 (GPIO2), U9.3 (GPIO25_D2)
- net CS 6: now reaches R7.2, U17.11 (GPIO18), U6.3 (GPIO25_D2)
- net CS 12: now reaches R13.2, U12.3 (GPIO25_D2), U17.30 (GPIO40)
- net CS 2: now reaches R3.2, U17.5 (GPIO5), U2.3 (GPIO25_D2)
- net CS 10: now reaches R11.2, U10.3 (GPIO25_D2), U17.28 (GPIO42)
- net CS 16: now reaches R16.2, U16.3 (GPIO25_D2), U17.16 (GPIO10)
- net CS 13: now reaches R14.2, U13.3 (GPIO25_D2), U17.31 (GPIO39)
- net CS 5: now reaches R6.2, U17.8 (GPIO15), U5.3 (GPIO25_D2)
- net CS 7: now reaches R8.2, U17.12 (GPIO8), U7.3 (GPIO25_D2)
- net CS 8: now reaches R9.2, U17.15 (GPIO9), U8.3 (GPIO25_D2)
- net CS 15: now reaches R17.2, U15.3 (GPIO25_D2), U17.20 (GPIO14)
- net CS 1: now reaches R2.2, U1.3 (GPIO25_D2), U17.4 (GPIO4)
- net CS 4: now reaches R5.2, U17.7 (GPIO7), U4.3 (GPIO25_D2)
Changed lines of the file:
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@@
 		)
 	)
+	(label "CS 5"
+		(at 21.59 203.2 0)
+		(effects
+			(font
+				(size 1.27 1.27)
+			)
+			(justify left bottom)
+		)
+	)
 	(label "MOSI"
 		(at 76.2 34.29 0)
@@
 		)
 	)
+	(label "CS 16"
+		(at 180.34 328.93 0)
+		(effects
+			(font
+				(size 1.27 1.27)
+			)
+			(justify left bottom)
+		)
+	)
 	(label "MISO"
 		(at 234.95 161.29 0)
@@
 		)
 	)
+	(label "CS 6"
+		(at 21.59 243.84 0)
+		(effects
+			(font
+				(size 1.27 1.27)
+			)
+			(justify left bottom)
+		)
+	)
 	(label "SCK"
 		(at 139.7 201.93 0)
@@
 		)
 	)
+	(label "CS 4"
+		(at 21.59 163.83 0)
+		(effects
+			(font
+				(size 1.27 1.27)
+			)
+			(justify left bottom)
+		)
+	)
 	(label "SCK"
 		(at 234.95 245.11 0)
@@
 		)
 	)
+	(label "CS 3"
+		(at 21.59 123.19 0)
+		(effects
+			(font
+				(size 1.27 1.27)
+			)
+			(justify left bottom)
+		)
+	)
 	(label "MOSI"
 		(at 234.95 34.29 0)
@@
 		)
 	)
+	(label "CS 8"
+		(at 21.59 328.93 0)
+		(effects
+			(font
+				(size 1.27 1.27)
+			)
+			(justify left bottom)
+		)
+	)
 	(label "MISO"
 		(at 234.95 241.3 0)
@@
 		)
 	)
+	(label "CS 11"
+		(at 180.34 123.19 0)
+		(effects
+			(font
+				(size 1.27 1.27)
+			)
+			(justify left bottom)
+		)
+	)
 	(label "MOSI"
 		(at 76.2 116.84 0)
@@
 		)
 	)
+	(label "CS 10"
+		(at 180.34 80.01 0)
+		(effects
+			(font
+				(size 1.27 1.27)
+			)
+			(justify left bottom)
+		)
+	)
 	(label "SCK"
 		(at 234.95 41.91 0)
@@
 		)
 	)
+	(label "CS 15"
+		(at 181.61 287.02 0)
+		(effects
+			(font
+				(size 1.27 1.27)
+			)
+			(justify left bottom)
+		)
+	)
 	(label "MOSI"
 		(at 234.95 237.49 0)
@@
 		)
 	)
+	(label "CS 12"
+		(at 180.34 163.83 0)
+		(effects
+			(font
+				(size 1.27 1.27)
+			)
+			(justify left bottom)
+		)
+	)
 	(label "GPS_RX"
 		(at 111.76 316.23 0)
@@
 		)
 	)
+	(label "MicroSD Card Breakout"
+		(at 123.19 194.31 0)
+		(effects
+			(font
+				(size 1.27 1.27)
+			)
+			(justify left bottom)
+		)
+	)
 	(label "SCK"
 		(at 114.3 339.09 0)
@@
 		)
 	)
+	(label "CS 2"
+		(at 21.59 78.74 0)
+		(effects
+			(font
+				(size 1.27 1.27)
+			)
+			(justify left bottom)
+		)
+	)
 	(label "SCK"
 		(at 234.95 204.47 0)
@@
 		)
 	)
+	(label "CS 13"
+		(at 180.34 203.2 0)
+		(effects
+			(font
+				(size 1.27 1.27)
+			)
+			(justify left bottom)
+		)
+	)
 	(label "MISO"
 		(at 236.22 284.48 0)
@@
 		)
 	)
+	(label "CS 7"
+		(at 22.86 287.02 0)
+		(effects
+			(font
+				(size 1.27 1.27)
+			)
+			(justify left bottom)
+		)
+	)
+	(label "CS 9"
+		(at 180.34 41.91 0)
+		(effects
+			(font
+				(size 1.27 1.27)
+			)
+			(justify left bottom)
+		)
+	)
 	(label "SCK"
 		(at 76.2 245.11 0)
@@
 		)
 	)
+	(label "CS 1"
+		(at 21.59 39.37 0)
+		(effects
+			(font
+				(size 1.27 1.27)
+			)
+			(justify left bottom)
+		)
+	)
 	(label "SCK"
 		(at 76.2 204.47 0)
@@
 		)
 	)
+	(label "CS 14"
+		(at 180.34 243.84 0)
+		(effects
+			(font
+				(size 1.27 1.27)
+			)
+			(justify left bottom)
+		)
+	)
 	(label "MISO"
 		(at 234.95 120.65 0)
@@
 		(dnp no)
 		(fields_autoplaced yes)
-		(property "Reference" "U19"
+		(property "Reference" "U18"
 			(at 132.08 218.44 0)
 			(show_name no)
@@
 			(project "pcb"
 				(path "/177b52ef-cce2-4dab-a936-75649664352c"
-					(reference "U19")
+					(reference "U18")
 					(unit 1)
 				)
@@
 		(dnp no)
 		(fields_autoplaced yes)
-		(property "Reference" "U15"
+		(property "Reference" "U16"
 			(at 208.28 302.26 0)
 			(show_name no)
@@
 			(project "pcb"
 				(path "/177b52ef-cce2-4dab-a936-75649664352c"
-					(reference "U15")
+					(reference "U16")
 					(unit 1)
 				)
@@
 		(in_pos_files yes)
 		(dnp no)
-		(fields_autoplaced yes)
-		(property "Reference" "U16"
-			(at 133.35 290.83 0)
+		(property "Reference" "U17"
+			(at 132.334 286.766 0)
 			(show_name no)
 			(do_not_autoplace no)
@@
 			)
 		)
-		(property "Value" ""
-			(at 121.92 293.37 0)
+		(property "Value" "ESP32-S3 DevKitC-A"
+			(at 132.588 291.084 0)
 			(show_name no)
 			(do_not_autoplace no)
@@
 			(project "pcb"
 				(path "/177b52ef-cce2-4dab-a936-75649664352c"
-					(reference "U16")
+					(reference "U17")
 					(unit 1)
 				)
@@
 		(dnp no)
 		(property "Reference" "J2"
-			(at 119.888 195.58 0)
+			(at 132.08 190.754 0)
 			(show_name no)
 			(do_not_autoplace no)
@@
 		)
 		(property "Value" "Conn_01x06_Pin"
-			(at 132.715 196.85 0)
+			(at 132.08 196.342 0)
 			(show_name no)
 			(do_not_autoplace no)
@@
 		(dnp no)
 		(fields_autoplaced yes)
-		(property "Reference" "U18"
+		(property "Reference" "U15"
 			(at 209.55 260.35 0)
 			(show_name no)
@@
 			(project "pcb"
 				(path "/177b52ef-cce2-4dab-a936-75649664352c"
-					(reference "U18")
+					(reference "U15")
 					(unit 1)
 				)

Commit message: Added net classes and colors, squared away controller footprint, sorted power input battery symbol
Parts:
- BT1: symbol Device:Battery -> esp32_wroom:Battery_-_POWER_OUTPUT
- J1: value Conn_01x04_Pin -> GPS Module Breakout
- J2: value Conn_01x06_Pin -> MicroSD Card Breakout
- U17: value ESP32-S3 DevKitC-A -> ESP32-S3 DevKitC-1
Connections:
- net +5V: now also U18.3 (VI)
- net GND: now also C1.1
Other:
- moved on the sheet: C1

Commit message: Add my 74HC125 for protecting the SPI lines from microsd card bus hogging
Parts:
- added C3: 100nF, Capacitor_THT:C_Disc_D5.0mm_W2.5mm_P2.50mm, symbol Device:C
- added U19: SN74HC125N, SN74HC125N:DIP794W45P254L1969H508Q14, symbol 74HC125:SN74HC125N
Connections:
- net CS 16 is gone; now on net CS 15: R16.2, U16.3 (GPIO25_D2), U17.16 (GPIO10)
- net CS 15: now also U17.38 (GPIO48)
- net GND: now also C3.1, U19.13 (4~OE), U19.7 (GND)
- net MISO: now also U19.3 (1Y); no longer J2.4 (Pin_4)
- net MOSI: now also U19.5 (2A); no longer J2.3 (Pin_3)
- net SCK: now also U19.9 (3A); no longer J2.2 (Pin_2)
- net at C2.2, U18.2 (VO): now also C3.2, U19.14 (VCC)
- net CS 0: now reaches R1.1, U17.26 (GPIO1)
- net CS 0: now also C2.1, J2.6 (Pin_6), R1.2, U19.1 (1~OE), U19.10 (3~OE), U19.12 (4A), U19.4 (2~OE); no longer J2.1 (Pin_1)
- new net: J2.1 (Pin_1), U19.11 (4Y)
- new net: J2.4 (Pin_4), U19.2 (1A)
- new net: J2.3 (Pin_3), U19.6 (2Y)
- new net: J2.2 (Pin_2), U19.8 (3Y)
Other:
- moved on the sheet: C1, C2, J1, J2, R1, R10, R11, R12, R13, R14, R15, R16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

Commit message: Add 74HC125 for SPI bus protection from microsd modules
Parts:
- U19: footprint SN74HC125N:DIP794W45P254L1969H508Q14 -> Package_DIP:DIP-14_W7.62mm_LongPads
Connections:
- net CS 15: no longer R16.2, U16.3 (GPIO25_D2), U17.16 (GPIO10), U17.38 (GPIO48)
- new net CS 16: R16.2, U16.3 (GPIO25_D2), U17.16 (GPIO10)
Changed lines of the file:
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@@
 	)
 	(junction
-		(at 220.98 359.41)
-		(diameter 0)
-		(color 0 0 0 0)
-	)
-	(junction
 		(at 87.63 337.82)
 		(diameter 0)
@@
 	)
 	(junction
-		(at 168.91 359.41)
-		(diameter 0)
-		(color 0 0 0 0)
-	)
-	(junction
 		(at 87.63 212.09)
 		(diameter 0)
@@
 	)
 	(junction
-		(at 167.64 334.01)
-		(diameter 0)
-		(color 0 0 0 0)
-	)
-	(junction
 		(at 87.63 252.73)
 		(diameter 0)
@@
 	(wire
 		(pts
-			(xy 168.91 359.41) (xy 220.98 359.41)
+			(xy 121.92 356.87) (xy 220.98 356.87)
 		)
 		(stroke
@@
 	(wire
 		(pts
-			(xy 121.92 344.17) (xy 121.92 359.41)
+			(xy 121.92 344.17) (xy 121.92 356.87)
 		)
 		(stroke
@@
 	(wire
 		(pts
-			(xy 220.98 359.41) (xy 223.52 359.41)
+			(xy 287.02 73.66) (xy 292.1 73.66)
 		)
 		(stroke
@@
 	(wire
 		(pts
-			(xy 287.02 73.66) (xy 292.1 73.66)
+			(xy 116.84 334.01) (xy 116.84 359.41)
 		)
 		(stroke
@@
 	(wire
 		(pts
-			(xy 167.64 334.01) (xy 168.91 334.01)
-		)
-		(stroke
-			(width 0)
-			(type default)
-		)
-	)
-	(wire
-		(pts
 			(xy 280.67 72.39) (xy 278.13 72.39)
 		)
@@
 	(wire
 		(pts
+			(xy 139.7 334.01) (xy 116.84 334.01)
+		)
+		(stroke
+			(width 0)
+			(type default)
+		)
+	)
+	(wire
+		(pts
 			(xy 220.98 293.37) (xy 227.33 293.37)
 		)
@@
 	(wire
 		(pts
-			(xy 168.91 334.01) (xy 168.91 359.41)
+			(xy 280.67 321.31) (xy 278.13 321.31)
 		)
 		(stroke
@@
 	(wire
 		(pts
-			(xy 280.67 321.31) (xy 278.13 321.31)
+			(xy 177.8 349.25) (xy 167.64 349.25)
 		)
 		(stroke
@@
 	(wire
 		(pts
-			(xy 177.8 349.25) (xy 167.64 349.25)
+			(xy 116.84 359.41) (xy 223.52 359.41)
 		)
 		(stroke
@@
 	(wire
 		(pts
-			(xy 139.7 334.01) (xy 167.64 334.01)
-		)
-		(stroke
-			(width 0)
-			(type default)
-		)
-	)
-	(wire
-		(pts
 			(xy 21.59 133.35) (xy 87.63 133.35)
 		)
@@
 	(wire
 		(pts
-			(xy 220.98 293.37) (xy 220.98 359.41)
+			(xy 220.98 293.37) (xy 220.98 356.87)
 		)
 		(stroke
@@
 	(wire
 		(pts
-			(xy 121.92 359.41) (xy 168.91 359.41)
-		)
-		(stroke
-			(width 0)
-			(type default)
-		)
-	)
-	(wire
-		(pts
 			(xy 142.24 26.67) (xy 142.24 25.4)
 		)
@@
 			)
 		)
-		(property "Footprint" "SN74HC125N:DIP794W45P254L1969H508Q14"
+		(property "Footprint" "Package_DIP:DIP-14_W7.62mm_LongPads"
 			(at 152.4 250.19 0)
 			(hide yes)

Commit message: Fix ERC warnings, place new components in PCB
Parts:
- added U20, U21: SN74HC138N, SN74HC138N:DIP794W45P254L1969H508Q16, symbol SN74HC138N:SN74HC138N
Connections:
- net +5V: now also U20.16 (VCC), U20.6 (G1), U21.16 (VCC)
- net CS 10: now also U21.14 (Y1); no longer U17.28 (GPIO42)
- net CS 11: now also U21.13 (Y2); no longer U17.29 (GPIO41)
- net CS 12: now also U21.12 (Y3); no longer U17.30 (GPIO40)
- net CS 13: now also U21.11 (Y4); no longer U17.31 (GPIO39)
- net CS 14: now also U21.10 (Y5); no longer U17.40 (GPIO21)
- net CS 15: now also U21.9 (Y6); no longer U17.20 (GPIO14)
- net CS 16: now also U21.7 (Y7); no longer U17.16 (GPIO10)
- net GND: now also U20.8 (GND), U21.4 (~{G2A}), U21.8 (GND)
- net CS 0 renamed CS 00
- net CS 00: now also U17.4 (GPIO4); no longer U17.26 (GPIO1)
- net CS 1 renamed CS 01
- net CS 01: now also U20.15 (Y0); no longer U17.4 (GPIO4)
- net CS 2 renamed CS 02
- net CS 02: now also U20.14 (Y1); no longer U17.5 (GPIO5)
- net CS 3 renamed CS 03
- net CS 03: now also U20.13 (Y2); no longer U17.6 (GPIO6)
- net CS 4 renamed CS 04
- net CS 04: now also U20.12 (Y3); no longer U17.7 (GPIO7)
- net CS 5 renamed CS 05
- net CS 05: now also U20.11 (Y4); no longer U17.8 (GPIO15)
- net CS 6 renamed CS 06
- net CS 06: now also U20.10 (Y5); no longer U17.11 (GPIO18)
- net CS 7 renamed CS 07
- net CS 07: now also U20.9 (Y6); no longer U17.12 (GPIO8)
- net CS 8 renamed CS 08
- net CS 08: now also U20.7 (Y7); no longer U17.15 (GPIO9)
- net CS 9 renamed CS 09
- net CS 09: now also U21.15 (Y0); no longer U17.27 (GPIO2)
- new net CS Addr 1: U17.5 (GPIO5), U20.1 (A), U21.1 (A)
- new net CS Addr 2: U17.6 (GPIO6), U20.2 (B), U21.2 (B)
- new net CS Addr 3: U17.7 (GPIO7), U20.3 (C), U21.3 (C)
- new net CS Bank Sel: U17.8 (GPIO15), U20.4 (~{G2A}), U21.6 (G1)
- new net CS ENABLE: U17.11 (GPIO18), U20.5 (~{G2B}), U21.5 (~{G2B})
- no-connect marks 132 -> 143
Other:
- moved on the sheet: BT1, C1, C2, C3, J1, J2, R1, U18, U19
